Commit message: succeed in launch

File: open_manipulator_x_robot/urdf/open_manipulator_x.ros2_control.xacro (robot description, xacro)
@@ -1,5 +1,5 @@
 <?xml version="1.0"?>
 <robot xmlns:xacro="http://www.ros.org/wiki/xacro">
-  <xacro:macro name="open_manipulator_x.ros2_control" params="name">
+  <xacro:macro name="open_manipulator_x_ros2_control" params="name">
     <ros2_control name="${name}" type="system">
       <hardware>

File: open_manipulator_x_robot/urdf/open_manipulator_x_robot.urdf.xacro (robot description, xacro)
@@ -5,5 +5,5 @@
   <xacro:include filename="$(find open_manipulator_x_robot)/urdf/open_manipulator_x.urdf.xacro" />
   <!-- Import ros2_control -->
-  <xacro:include filename="$(find open_manipulator_x_robot)/urdf/open_manipulator_x.ros2_control.urdf.xacro" />
+  <xacro:include filename="$(find open_manipulator_x_robot)/urdf/open_manipulator_x.ros2_control.xacro" />
   <!-- World -->
   <link name="world"/>
