Commit message: refine xacro

File: open_manipulator_x_robot/urdf/open_manipulator_x.xacro (robot description, xacro)
@@ -220,35 +220,4 @@
     </inertial>
   </link>
-  <!-- end effector joint -->
-  <joint name="end_effector_joint" type="fixed">
-    <origin xyz="0.126 0.0 0.0" rpy="0 0 0"/>
-    <parent link="link5"/>
-    <child link="end_effector_link"/>
-  </joint>
-  <!-- end effector link -->
-  <link name="end_effector_link">
-    <visual>
-      <origin xyz="0 0 0" rpy="0 0 0"/>
-      <geometry>
-        <box size="0.01 0.01 0.01" />
-      </geometry>
-      <material name="red"/>
-     </visual>
-    <inertial>
-      <origin xyz="0 0 0" />
-      <mass value="1.0e-03" />
-      <inertia ixx="1.0e-03" ixy="0.0" ixz="0.0"
-               iyy="1.0e-03" iyz="0.0"
-               izz="1.0e-03" />
-    </inertial>
-  </link>
-  <!-- Realsense Camera Joint Position -->
-  <joint name="camera_joint" type="fixed">
-    <axis xyz="0 1 0" />
-    <origin xyz="0.070 0.032 0.052" rpy="0 0 0"/>
-    <parent link="link5"/>
-    <child link="camera_link"/>
-  </joint>
-  <link name="camera_link"/>
 </xacro:macro>
 </robot>

File: open_manipulator_x_robot/urdf/open_manipulator_x_robot.urdf.xacro (robot description, xacro)
@@ -1,13 +1,10 @@
 <?xml version="1.0"?>
-<!-- OpenManipulator Chain -->
 <robot name="open_manipulator_x" xmlns:xacro="http://ros.org/wiki/xacro">
-  <!-- Import URDF -->
-  <xacro:include filename="$(find open_manipulator_x_robot)/urdf/open_manipulator_x.urdf.xacro" />
-  <!-- Import ros2_control -->
+  <xacro:include filename="$(find open_manipulator_x_robot)/urdf/open_manipulator_x.xacro" />
   <xacro:include filename="$(find open_manipulator_x_robot)/urdf/open_manipulator_x.ros2_control.xacro" />
-  <!-- World -->
   <link name="world"/>
   <xacro:open_manipulator_x parent="world">
     <origin xyz="0 0 0" rpy="0 0 0" />
   </xacro:open_manipulator_x>
+  <xacro:open_manipulator_x_ros2_control name="open_manipulator_x_ros2_control" />
 </robot>
