Commit message: rename to pan_tilt_bot

File: pan_tilt_bot_robot/urdf/pan_tilt_bot.ros2_control.xacro (robot description, xacro)
@@ -1,5 +1,5 @@
 <?xml version="1.0"?>
 <robot xmlns:xacro="http://www.ros.org/wiki/xacro">
-  <xacro:macro name="pan_tilt_ros2_control" params="name">
+  <xacro:macro name="pan_tilt_bot_ros2_control" params="name">
     <ros2_control name="${name}" type="system">
       <hardware>

File: pan_tilt_bot_robot/urdf/pan_tilt_bot.xacro (robot description, xacro)
@@ -2,6 +2,6 @@
 <robot xmlns:xacro="http://ros.org/wiki/xacro">
 <!-- Import Rviz colors -->
-<xacro:include filename="$(find pan_tilt_robot)/urdf/pan_tilt.material.xacro" />
-<xacro:macro name="pan_tilt" params="parent *origin">
+<xacro:include filename="$(find pan_tilt_bot_robot)/urdf/pan_tilt_bot.material.xacro" />
+<xacro:macro name="pan_tilt_bot" params="parent *origin">
   <joint name="origin_to_link1" type="fixed">
     <xacro:insert_block name="origin" />
