Commit message: import meshes

File: pan_tilt_bot_robot/urdf/pan_tilt_bot.xacro (robot description, xacro)
@@ -1,98 +1,112 @@
 <?xml version="1.0"?>
 <robot xmlns:xacro="http://ros.org/wiki/xacro">
-<!-- Import Rviz colors -->
-<xacro:include filename="$(find pan_tilt_bot_robot)/urdf/pan_tilt_bot.material.xacro" />
-<xacro:macro name="pan_tilt_bot" params="parent *origin">
-  <joint name="origin_to_link1" type="fixed">
-    <xacro:insert_block name="origin" />
-    <parent link="${parent}" />
-    <child link="link1" />
-    <axis xyz="0 0 1" />
-  </joint>
-  <!-- Link 1 -->
-  <link name="link1">
-    <visual>
-      <origin xyz="0 0 0" rpy="0 0 0"/>
-      <geometry>
-        <mesh filename="package://open_manipulator_x_robot/meshes/chain_link1.stl" scale="0.001 0.001 0.001"/>
-      </geometry>
-      <material name="grey"/>
-    </visual>
-    <collision>
-      <origin xyz="0 0 0" rpy="0 0 0"/>
-      <geometry>
-        <mesh filename="package://open_manipulator_x_robot/meshes/chain_link1.stl" scale="0.001 0.001 0.001"/>
-      </geometry>
-    </collision>
-    <inertial>
-      <origin xyz="3.0876154e-04 0.0000000e+00 -1.2176461e-04" />
-      <mass value="7.9119962e-02" />
-      <inertia ixx="1.2505234e-05" ixy="0.0" ixz="-1.7855208e-07"
-               iyy="2.1898364e-05" iyz="0.0"
-               izz="1.9267361e-05" />
-    </inertial>
-  </link>
-  <!-- Joint 1 -->
-  <joint name="joint1" type="revolute">
-    <parent link="link1"/>
-    <child link="link2"/>
-    <origin xyz="0.012 0.0 0.017" rpy="0 0 0"/>
-    <axis xyz="0 0 1"/>
-    <limit velocity="4.8" effort="1" lower="-2.82743338823" upper="2.82743338823" />
-  </joint>
-  <!--  Link 2 -->
-  <link name="link2">
-    <visual>
-      <origin xyz="0 0 0.019" rpy="0 0 0"/>
-      <geometry>
-        <mesh filename="package://open_manipulator_x_robot/meshes/chain_link2.stl" scale="0.001 0.001 0.001"/>
-      </geometry>
-      <material name="grey"/>
-    </visual>
-    <collision>
-      <origin xyz="0 0 0.019" rpy="0 0 0"/>
-      <geometry>
-        <mesh filename="package://open_manipulator_x_robot/meshes/chain_link2.stl" scale="0.001 0.001 0.001"/>
-      </geometry>
-    </collision>
-     <inertial>
-      <origin xyz="-3.0184870e-04 5.4043684e-04 0.047433464e-02" />
-      <mass value="9.8406837e-02" />
-      <inertia ixx="3.4543422e-05" ixy="-1.6031095e-08" ixz="-3.8375155e-07"
-               iyy="3.2689329e-05" iyz="2.8511935e-08"
-               izz="1.8850320e-05" />
-    </inertial>
-  </link>
-  <!--  Joint 2 -->
-  <joint name="joint2" type="revolute">
-    <parent link="link2"/>
-    <child link="link3"/>
-    <origin xyz="0.0 0.0 0.0595" rpy="0 0 0"/>
-    <axis xyz="0 1 0"/>
-    <limit velocity="4.8" effort="1" lower="-1.79070781255" upper="1.57079632679" />
-  </joint>
-  <!--  Link 3 -->
-  <link name="link3">
-    <visual>
-      <origin xyz="0 0 0" rpy="0 0 0"/>
-      <geometry>
-        <mesh filename="package://open_manipulator_x_robot/meshes/chain_link3.stl" scale="0.001 0.001 0.001"/>
-      </geometry>
-      <material name="grey"/>
-    </visual>
-    <collision>
-      <origin xyz="0 0 0" rpy="0 0 0"/>
-      <geometry>
-        <mesh filename="package://open_manipulator_x_robot/meshes/chain_link3.stl" scale="0.001 0.001 0.001"/>
-      </geometry>
-    </collision>
-    <inertial>
-      <origin xyz="1.0308393e-02 3.7743363e-04 1.0170197e-01" />
-      <mass value="1.3850917e-01" />
-      <inertia ixx="3.3055381e-04" ixy="-9.7940978e-08" ixz="-3.8505711e-05"
-               iyy="3.4290447e-04" iyz="-1.5717516e-06"
-               izz="6.0346498e-05" />
-    </inertial>
-  </link>
-</xacro:macro>
+  <!-- Import Rviz colors -->
+  <xacro:include filename="$(find pan_tilt_bot_robot)/urdf/pan_tilt_bot.material.xacro" />
+  <xacro:macro name="pan_tilt_bot" params="parent *origin">
+    <link name="j1_link">
+      <inertial>
+        <origin rpy="0 0 0" xyz="-5.549338143508866e-15 0.011937164947263951 0.019605935309866387"/>
+        <mass value="0.34009000706899195"/>
+        <inertia ixx="9.4e-05" ixy="-0.0" ixz="0.0" iyy="5.5e-05" iyz="0.0" izz="8.2e-05"/>
+      </inertial>
+      <visual>
+        <origin rpy="0 0 0" xyz="0 0 0"/>
+        <geometry>
+          <mesh filename="package://pan_tilt_bot_robot/meshes/j1.stl" scale="0.001 0.001 0.001"/>
+        </geometry>
+        <material name="grey"/>
+      </visual>
+      <collision>
+        <origin rpy="0 0 0" xyz="0 0 0"/>
+        <geometry>
+          <mesh filename="package://pan_tilt_bot_robot/meshes/j1.stl" scale="0.001 0.001 0.001"/>
+        </geometry>
+      </collision>
+    </link>
+    <link name="j1_horn_link">
+      <inertial>
+        <origin rpy="0 0 0" xyz="7.323601717155284e-17 -3.584248942771506e-07 0.0027880990797749597"/>
+        <mass value="0.016309929358964557"/>
+        <inertia ixx="3e-06" ixy="-0.0" ixz="-0.0" iyy="1e-06" iyz="0.0" izz="4e-06"/>
+      </inertial>
+      <visual>
+        <origin rpy="0 0 0" xyz="0.0 -0.000319 -0.038"/>
+        <geometry>
+          <mesh filename="package://pan_tilt_bot_robot/meshes/j1_horn.stl" scale="0.001 0.001 0.001"/>
+        </geometry>
+        <material name="grey"/>
+      </visual>
+      <collision>
+        <origin rpy="0 0 0" xyz="0.0 -0.000319 -0.038"/>
+        <geometry>
+          <mesh filename="package://pan_tilt_bot_robot/meshes/j1_horn.stl" scale="0.001 0.001 0.001"/>
+        </geometry>
+      </collision>
+    </link>
+    <link name="j2_link">
+      <inertial>
+        <origin rpy="0 0 0" xyz="-0.010999999999994571 0.016393706265213467 0.02038147662781581"/>
+        <mass value="0.34009000706899195"/>
+        <inertia ixx="9.4e-05" ixy="0.0" ixz="-0.0" iyy="8.2e-05" iyz="0.0" izz="5.5e-05"/>
+      </inertial>
+      <visual>
+        <origin rpy="0 0 0" xyz="-0.011 0.016681 -0.0465"/>
+        <geometry>
+          <mesh filename="package://pan_tilt_bot_robot/meshes/j2.stl" scale="0.001 0.001 0.001"/>
+        </geometry>
+        <material name="grey"/>
+      </visual>
+      <collision>
+        <origin rpy="0 0 0" xyz="-0.011 0.016681 -0.0465"/>
+        <geometry>
+          <mesh filename="package://pan_tilt_bot_robot/meshes/j2.stl" scale="0.001 0.001 0.001"/>
+        </geometry>
+      </collision>
+    </link>
+    <link name="j2_horn_link">
+      <inertial>
+        <origin rpy="0 0 0" xyz="7.674625448279525e-16 -0.019000358424909176 0.03767262835995369"/>
+        <mass value="0.05331898839844395"/>
+        <inertia ixx="3.2e-05" ixy="-0.0" ixz="0.0" iyy="2e-05" iyz="-0.0" izz="1.9e-05"/>
+      </inertial>
+      <visual>
+        <origin rpy="0 0 0" xyz="-0.0 -0.019319 -0.0785"/>
+        <geometry>
+          <mesh filename="package://pan_tilt_bot_robot/meshes/j2_horn.stl" scale="0.001 0.001 0.001"/>
+        </geometry>
+        <material name="grey"/>
+      </visual>
+      <collision>
+        <origin rpy="0 0 0" xyz="-0.0 -0.019319 -0.0785"/>
+        <geometry>
+          <mesh filename="package://pan_tilt_bot_robot/meshes/j2_horn.stl" scale="0.001 0.001 0.001"/>
+        </geometry>
+      </collision>
+    </link>
+    <joint name="origin_to_j1" type="fixed">
+      <xacro:insert_block name="origin" />
+      <parent link="${parent}" />
+      <child link="j1_link" />
+      <axis xyz="0 0 1" />
+    </joint>
+    <joint name="j1" type="revolute">
+      <origin rpy="0 0 0" xyz="0.0 0.000319 0.038"/>
+      <parent link="j1_link"/>
+      <child link="j1_horn_link"/>
+      <axis xyz="-0.0 -0.0 -1.0"/>
+      <limit effort="100" lower="-2.96706" upper="2.96706" velocity="100"/>
+    </joint>
+    <joint name="j1_horn_to_j2" type="fixed">
+      <origin rpy="0 0 0" xyz="0.011 -0.017 0.0085"/>
+      <parent link="j1_horn_link"/>
+      <child link="j2_link"/>
+    </joint>
+    <joint name="j2" type="revolute">
+      <origin rpy="0 0 0" xyz="-0.011 0.036 0.032"/>
+      <parent link="j2_link"/>
+      <child link="j2_horn_link"/>
+      <axis xyz="-0.0 -1.0 -0.0"/>
+      <limit effort="100" lower="-1.745329" upper="1.745329" velocity="100"/>
+    </joint>
+  </xacro:macro>
 </robot>

Commit message: attach d435

File: pan_tilt_bot_robot/urdf/pan_tilt_bot.xacro (robot description, xacro)
@@ -91,5 +91,5 @@
     </joint>
     <joint name="j1" type="revolute">
-      <origin rpy="0 0 0" xyz="0.0 0.000319 0.038"/>
+      <origin rpy="0 0 1.5708" xyz="0.0 0.000319 0.038"/>
       <parent link="j1_link"/>
       <child link="j1_horn_link"/>
@@ -107,5 +107,5 @@
       <child link="j2_horn_link"/>
       <axis xyz="-0.0 -1.0 -0.0"/>
-      <limit effort="100" lower="-1.745329" upper="1.745329" velocity="100"/>
+      <limit effort="100" lower="-2.1" upper="2.1" velocity="100"/>
     </joint>
   </xacro:macro>

File: pan_tilt_bot_robot/urdf/pan_tilt_bot_robot.urdf.xacro (robot description, xacro)
@@ -3,8 +3,12 @@
   <xacro:include filename="$(find pan_tilt_bot_robot)/urdf/pan_tilt_bot.xacro" />
   <xacro:include filename="$(find pan_tilt_bot_robot)/urdf/pan_tilt_bot.ros2_control.xacro" />
+  <xacro:include filename="$(find realsense2_description)/urdf/_d435.urdf.xacro" />
   <link name="world"/>
   <xacro:pan_tilt_bot parent="world">
     <origin xyz="0 0 0" rpy="0 0 0" />
   </xacro:pan_tilt_bot>
+  <xacro:sensor_d435 parent="j2_horn_link" use_nominal_extrinsics="true" add_plug="false">
+    <origin xyz="0.0125 -0.019 0.065" rpy="0 -1.5708 0"/>
+  </xacro:sensor_d435>
   <xacro:pan_tilt_bot_ros2_control name="pan_tilt_bot_ros2_control" />
 </robot>
