Commit message: rename to pantilt_bot

File: pantilt_bot_robot/urdf/pantilt_bot.ros2_control.xacro (robot description, xacro)
@@ -1,5 +1,5 @@
 <?xml version="1.0"?>
 <robot xmlns:xacro="http://www.ros.org/wiki/xacro">
-  <xacro:macro name="pan_tilt_bot_ros2_control" params="name">
+  <xacro:macro name="pantilt_bot_ros2_control" params="name">
     <ros2_control name="${name}" type="system">
       <hardware>

File: pantilt_bot_robot/urdf/pantilt_bot.xacro (robot description, xacro)
@@ -2,6 +2,6 @@
 <robot xmlns:xacro="http://ros.org/wiki/xacro">
   <!-- Import Rviz colors -->
-  <xacro:include filename="$(find pan_tilt_bot_robot)/urdf/pan_tilt_bot.material.xacro" />
-  <xacro:macro name="pan_tilt_bot" params="parent *origin">
+  <xacro:include filename="$(find pantilt_bot_robot)/urdf/pantilt_bot.material.xacro" />
+  <xacro:macro name="pantilt_bot" params="parent *origin">
     <link name="j1_link">
       <inertial>
@@ -13,5 +13,5 @@
         <origin rpy="0 0 0" xyz="0 0 0"/>
         <geometry>
-          <mesh filename="package://pan_tilt_bot_robot/meshes/j1.stl" scale="0.001 0.001 0.001"/>
+          <mesh filename="package://pantilt_bot_robot/meshes/j1.stl" scale="0.001 0.001 0.001"/>
         </geometry>
         <material name="grey"/>
@@ -20,5 +20,5 @@
         <origin rpy="0 0 0" xyz="0 0 0"/>
         <geometry>
-          <mesh filename="package://pan_tilt_bot_robot/meshes/j1.stl" scale="0.001 0.001 0.001"/>
+          <mesh filename="package://pantilt_bot_robot/meshes/j1.stl" scale="0.001 0.001 0.001"/>
         </geometry>
       </collision>
@@ -33,5 +33,5 @@
         <origin rpy="0 0 0" xyz="0.0 -0.000319 -0.038"/>
         <geometry>
-          <mesh filename="package://pan_tilt_bot_robot/meshes/j1_horn.stl" scale="0.001 0.001 0.001"/>
+          <mesh filename="package://pantilt_bot_robot/meshes/j1_horn.stl" scale="0.001 0.001 0.001"/>
         </geometry>
         <material name="grey"/>
@@ -40,5 +40,5 @@
         <origin rpy="0 0 0" xyz="0.0 -0.000319 -0.038"/>
         <geometry>
-          <mesh filename="package://pan_tilt_bot_robot/meshes/j1_horn.stl" scale="0.001 0.001 0.001"/>
+          <mesh filename="package://pantilt_bot_robot/meshes/j1_horn.stl" scale="0.001 0.001 0.001"/>
         </geometry>
       </collision>
@@ -53,5 +53,5 @@
         <origin rpy="0 0 0" xyz="-0.011 0.016681 -0.0465"/>
         <geometry>
-          <mesh filename="package://pan_tilt_bot_robot/meshes/j2.stl" scale="0.001 0.001 0.001"/>
+          <mesh filename="package://pantilt_bot_robot/meshes/j2.stl" scale="0.001 0.001 0.001"/>
         </geometry>
         <material name="grey"/>
@@ -60,5 +60,5 @@
         <origin rpy="0 0 0" xyz="-0.011 0.016681 -0.0465"/>
         <geometry>
-          <mesh filename="package://pan_tilt_bot_robot/meshes/j2.stl" scale="0.001 0.001 0.001"/>
+          <mesh filename="package://pantilt_bot_robot/meshes/j2.stl" scale="0.001 0.001 0.001"/>
         </geometry>
       </collision>
@@ -73,5 +73,5 @@
         <origin rpy="0 0 0" xyz="-0.0 -0.019319 -0.0785"/>
         <geometry>
-          <mesh filename="package://pan_tilt_bot_robot/meshes/j2_horn.stl" scale="0.001 0.001 0.001"/>
+          <mesh filename="package://pantilt_bot_robot/meshes/j2_horn.stl" scale="0.001 0.001 0.001"/>
         </geometry>
         <material name="grey"/>
@@ -80,5 +80,5 @@
         <origin rpy="0 0 0" xyz="-0.0 -0.019319 -0.0785"/>
         <geometry>
-          <mesh filename="package://pan_tilt_bot_robot/meshes/j2_horn.stl" scale="0.001 0.001 0.001"/>
+          <mesh filename="package://pantilt_bot_robot/meshes/j2_horn.stl" scale="0.001 0.001 0.001"/>
         </geometry>
       </collision>
