Commit message: rename joint names

File: pantilt_bot_description/urdf/pantilt_bot.ros2_control.xacro (robot description, xacro)
@@ -7,5 +7,5 @@
         <param name="usb_port">/dev/ttyUSB0</param>
         <param name="baud_rate">1000000</param>
-        <param name="joint_ids">11,12,13,14,15</param>
+        <param name="joint_ids">11,12</param>
         <param name="use_dummy">true</param>
       </hardware>

File: pantilt_bot_description/urdf/pantilt_bot.urdf.xacro (robot description, xacro)
@@ -8,5 +8,5 @@
     <origin xyz="0 0 0" rpy="0 0 0" />
   </xacro:pantilt_bot>
-  <xacro:sensor_d435 parent="j2_horn_link" use_nominal_extrinsics="true" add_plug="false">
+  <xacro:sensor_d435 parent="joint2_horn_link" use_nominal_extrinsics="true" add_plug="false">
     <origin xyz="0.0125 -0.019 0.065" rpy="0 -1.5708 0"/>
   </xacro:sensor_d435>

File: pantilt_bot_description/urdf/pantilt_bot.xacro (robot description, xacro)
@@ -4,5 +4,5 @@
   <xacro:include filename="$(find pantilt_bot_description)/urdf/pantilt_bot.material.xacro" />
   <xacro:macro name="pantilt_bot" params="parent *origin">
-    <link name="j1_link">
+    <link name="joint1_link">
       <inertial>
         <origin rpy="0 0 0" xyz="-5.549338143508866e-15 0.011937164947263951 0.019605935309866387"/>
@@ -13,5 +13,5 @@
         <origin rpy="0 0 0" xyz="0 0 0"/>
         <geometry>
-          <mesh filename="package://pantilt_bot_description/meshes/j1.stl" scale="0.001 0.001 0.001"/>
+          <mesh filename="package://pantilt_bot_description/meshes/joint1.stl" scale="0.001 0.001 0.001"/>
         </geometry>
         <material name="grey"/>
@@ -20,9 +20,9 @@
         <origin rpy="0 0 0" xyz="0 0 0"/>
         <geometry>
-          <mesh filename="package://pantilt_bot_description/meshes/j1.stl" scale="0.001 0.001 0.001"/>
+          <mesh filename="package://pantilt_bot_description/meshes/joint1.stl" scale="0.001 0.001 0.001"/>
         </geometry>
       </collision>
     </link>
-    <link name="j1_horn_link">
+    <link name="joint1_horn_link">
       <inertial>
         <origin rpy="0 0 0" xyz="7.323601717155284e-17 -3.584248942771506e-07 0.0027880990797749597"/>
@@ -33,5 +33,5 @@
         <origin rpy="0 0 0" xyz="0.0 -0.000319 -0.038"/>
         <geometry>
-          <mesh filename="package://pantilt_bot_description/meshes/j1_horn.stl" scale="0.001 0.001 0.001"/>
+          <mesh filename="package://pantilt_bot_description/meshes/joint1_horn.stl" scale="0.001 0.001 0.001"/>
         </geometry>
         <material name="grey"/>
@@ -40,9 +40,9 @@
         <origin rpy="0 0 0" xyz="0.0 -0.000319 -0.038"/>
         <geometry>
-          <mesh filename="package://pantilt_bot_description/meshes/j1_horn.stl" scale="0.001 0.001 0.001"/>
+          <mesh filename="package://pantilt_bot_description/meshes/joint1_horn.stl" scale="0.001 0.001 0.001"/>
         </geometry>
       </collision>
     </link>
-    <link name="j2_link">
+    <link name="joint2_link">
       <inertial>
         <origin rpy="0 0 0" xyz="-0.010999999999994571 0.016393706265213467 0.02038147662781581"/>
@@ -53,5 +53,5 @@
         <origin rpy="0 0 0" xyz="-0.011 0.016681 -0.0465"/>
         <geometry>
-          <mesh filename="package://pantilt_bot_description/meshes/j2.stl" scale="0.001 0.001 0.001"/>
+          <mesh filename="package://pantilt_bot_description/meshes/joint2.stl" scale="0.001 0.001 0.001"/>
         </geometry>
         <material name="grey"/>
@@ -60,9 +60,9 @@
         <origin rpy="0 0 0" xyz="-0.011 0.016681 -0.0465"/>
         <geometry>
-          <mesh filename="package://pantilt_bot_description/meshes/j2.stl" scale="0.001 0.001 0.001"/>
+          <mesh filename="package://pantilt_bot_description/meshes/joint2.stl" scale="0.001 0.001 0.001"/>
         </geometry>
       </collision>
     </link>
-    <link name="j2_horn_link">
+    <link name="joint2_horn_link">
       <inertial>
         <origin rpy="0 0 0" xyz="7.674625448279525e-16 -0.019000358424909176 0.03767262835995369"/>
@@ -73,5 +73,5 @@
         <origin rpy="0 0 0" xyz="-0.0 -0.019319 -0.0785"/>
         <geometry>
-          <mesh filename="package://pantilt_bot_description/meshes/j2_horn.stl" scale="0.001 0.001 0.001"/>
+          <mesh filename="package://pantilt_bot_description/meshes/joint2_horn.stl" scale="0.001 0.001 0.001"/>
         </geometry>
         <material name="grey"/>
@@ -80,30 +80,30 @@
         <origin rpy="0 0 0" xyz="-0.0 -0.019319 -0.0785"/>
         <geometry>
-          <mesh filename="package://pantilt_bot_description/meshes/j2_horn.stl" scale="0.001 0.001 0.001"/>
+          <mesh filename="package://pantilt_bot_description/meshes/joint2_horn.stl" scale="0.001 0.001 0.001"/>
         </geometry>
       </collision>
     </link>
-    <joint name="origin_to_j1" type="fixed">
+    <joint name="origin_to_joint1" type="fixed">
       <xacro:insert_block name="origin" />
       <parent link="${parent}" />
-      <child link="j1_link" />
+      <child link="joint1_link" />
       <axis xyz="0 0 1" />
     </joint>
-    <joint name="j1" type="revolute">
+    <joint name="joint1" type="revolute">
       <origin rpy="0 0 1.5708" xyz="0.0 0.000319 0.038"/>
-      <parent link="j1_link"/>
-      <child link="j1_horn_link"/>
+      <parent link="joint1_link"/>
+      <child link="joint1_horn_link"/>
       <axis xyz="-0.0 -0.0 -1.0"/>
       <limit effort="100" lower="-2.96706" upper="2.96706" velocity="100"/>
     </joint>
-    <joint name="j1_horn_to_j2" type="fixed">
+    <joint name="joint1_horn_to_joint2" type="fixed">
       <origin rpy="0 0 0" xyz="0.011 -0.017 0.0085"/>
-      <parent link="j1_horn_link"/>
-      <child link="j2_link"/>
+      <parent link="joint1_horn_link"/>
+      <child link="joint2_link"/>
     </joint>
-    <joint name="j2" type="revolute">
+    <joint name="joint2" type="revolute">
       <origin rpy="0 0 0" xyz="-0.011 0.036 0.032"/>
-      <parent link="j2_link"/>
-      <child link="j2_horn_link"/>
+      <parent link="joint2_link"/>
+      <child link="joint2_horn_link"/>
       <axis xyz="-0.0 -1.0 -0.0"/>
       <limit effort="100" lower="-2.1" upper="2.1" velocity="100"/>
