Commit message: change to _description

File: pantilt_bot_description/urdf/pantilt_bot.urdf.xacro (robot description, xacro)
@@ -1,6 +1,6 @@
 <?xml version="1.0"?>
 <robot name="pantilt_bot" xmlns:xacro="http://ros.org/wiki/xacro">
-  <xacro:include filename="$(find pantilt_bot_robot)/urdf/pantilt_bot.xacro" />
-  <xacro:include filename="$(find pantilt_bot_robot)/urdf/pantilt_bot.ros2_control.xacro" />
+  <xacro:include filename="$(find pantilt_bot_description)/urdf/pantilt_bot.xacro" />
+  <xacro:include filename="$(find pantilt_bot_description)/urdf/pantilt_bot.ros2_control.xacro" />
   <xacro:include filename="$(find realsense2_description)/urdf/_d435.urdf.xacro" />
   <link name="world"/>

File: pantilt_bot_description/urdf/pantilt_bot.xacro (robot description, xacro)
@@ -2,5 +2,5 @@
 <robot xmlns:xacro="http://ros.org/wiki/xacro">
   <!-- Import Rviz colors -->
-  <xacro:include filename="$(find pantilt_bot_robot)/urdf/pantilt_bot.material.xacro" />
+  <xacro:include filename="$(find pantilt_bot_description)/urdf/pantilt_bot.material.xacro" />
   <xacro:macro name="pantilt_bot" params="parent *origin">
     <link name="j1_link">
@@ -13,5 +13,5 @@
         <origin rpy="0 0 0" xyz="0 0 0"/>
         <geometry>
-          <mesh filename="package://pantilt_bot_robot/meshes/j1.stl" scale="0.001 0.001 0.001"/>
+          <mesh filename="package://pantilt_bot_description/meshes/j1.stl" scale="0.001 0.001 0.001"/>
         </geometry>
         <material name="grey"/>
@@ -20,5 +20,5 @@
         <origin rpy="0 0 0" xyz="0 0 0"/>
         <geometry>
-          <mesh filename="package://pantilt_bot_robot/meshes/j1.stl" scale="0.001 0.001 0.001"/>
+          <mesh filename="package://pantilt_bot_description/meshes/j1.stl" scale="0.001 0.001 0.001"/>
         </geometry>
       </collision>
@@ -33,5 +33,5 @@
         <origin rpy="0 0 0" xyz="0.0 -0.000319 -0.038"/>
         <geometry>
-          <mesh filename="package://pantilt_bot_robot/meshes/j1_horn.stl" scale="0.001 0.001 0.001"/>
+          <mesh filename="package://pantilt_bot_description/meshes/j1_horn.stl" scale="0.001 0.001 0.001"/>
         </geometry>
         <material name="grey"/>
@@ -40,5 +40,5 @@
         <origin rpy="0 0 0" xyz="0.0 -0.000319 -0.038"/>
         <geometry>
-          <mesh filename="package://pantilt_bot_robot/meshes/j1_horn.stl" scale="0.001 0.001 0.001"/>
+          <mesh filename="package://pantilt_bot_description/meshes/j1_horn.stl" scale="0.001 0.001 0.001"/>
         </geometry>
       </collision>
@@ -53,5 +53,5 @@
         <origin rpy="0 0 0" xyz="-0.011 0.016681 -0.0465"/>
         <geometry>
-          <mesh filename="package://pantilt_bot_robot/meshes/j2.stl" scale="0.001 0.001 0.001"/>
+          <mesh filename="package://pantilt_bot_description/meshes/j2.stl" scale="0.001 0.001 0.001"/>
         </geometry>
         <material name="grey"/>
@@ -60,5 +60,5 @@
         <origin rpy="0 0 0" xyz="-0.011 0.016681 -0.0465"/>
         <geometry>
-          <mesh filename="package://pantilt_bot_robot/meshes/j2.stl" scale="0.001 0.001 0.001"/>
+          <mesh filename="package://pantilt_bot_description/meshes/j2.stl" scale="0.001 0.001 0.001"/>
         </geometry>
       </collision>
@@ -73,5 +73,5 @@
         <origin rpy="0 0 0" xyz="-0.0 -0.019319 -0.0785"/>
         <geometry>
-          <mesh filename="package://pantilt_bot_robot/meshes/j2_horn.stl" scale="0.001 0.001 0.001"/>
+          <mesh filename="package://pantilt_bot_description/meshes/j2_horn.stl" scale="0.001 0.001 0.001"/>
         </geometry>
         <material name="grey"/>
@@ -80,5 +80,5 @@
         <origin rpy="0 0 0" xyz="-0.0 -0.019319 -0.0785"/>
         <geometry>
-          <mesh filename="package://pantilt_bot_robot/meshes/j2_horn.stl" scale="0.001 0.001 0.001"/>
+          <mesh filename="package://pantilt_bot_description/meshes/j2_horn.stl" scale="0.001 0.001 0.001"/>
         </geometry>
       </collision>

Commit message: fix realsense angle

File: pantilt_bot_description/urdf/pantilt_bot.urdf.xacro (robot description, xacro)
@@ -9,5 +9,5 @@
   </xacro:pantilt_bot>
   <xacro:sensor_d435 parent="joint2_horn_link" use_nominal_extrinsics="true" add_plug="false">
-    <origin xyz="0.0125 -0.019 0.065" rpy="0 -1.5708 0"/>
+    <origin xyz="-0.0125 -0.019 0.065" rpy="0 -1.5708 3.1416"/>
   </xacro:sensor_d435>
   <xacro:pantilt_bot_ros2_control name="pantilt_bot_ros2_control" />
