Commit message: fix joint1 axis

File: pantilt_bot_description/urdf/pantilt_bot.xacro (robot description, xacro)
@@ -94,5 +94,5 @@
       <parent link="joint1_link"/>
       <child link="joint1_horn_link"/>
-      <axis xyz="-0.0 -0.0 -1.0"/>
+      <axis xyz="-0.0 -0.0 1.0"/>
       <limit effort="100" lower="-2.96706" upper="2.96706" velocity="100"/>
     </joint>

Commit message: fix limit

File: pantilt_bot_description/urdf/pantilt_bot.xacro (robot description, xacro)
@@ -95,5 +95,5 @@
       <child link="joint1_horn_link"/>
       <axis xyz="-0.0 -0.0 1.0"/>
-      <limit effort="100" lower="-2.96706" upper="2.96706" velocity="100"/>
+      <limit effort="1" lower="-2.96706" upper="2.96706" velocity="${46 / 60.0 * 2.0 * pi}"/>
     </joint>
     <joint name="joint1_horn_to_joint2" type="fixed">
@@ -107,5 +107,5 @@
       <child link="joint2_horn_link"/>
       <axis xyz="-0.0 -1.0 -0.0"/>
-      <limit effort="100" lower="-2.1" upper="2.1" velocity="100"/>
+      <limit effort="1" lower="-2.1" upper="2.1" velocity="${46 / 60.0 * 2.0 * pi}"/>
     </joint>
   </xacro:macro>

Commit message: remove axis

File: pantilt_bot_description/urdf/pantilt_bot.xacro (robot description, xacro)
@@ -88,5 +88,4 @@
       <parent link="${parent}" />
       <child link="joint1_link" />
-      <axis xyz="0 0 1" />
     </joint>
     <joint name="joint1" type="revolute">
